Commit message: created mujoco demo with kuka

File: robots/trifinger/nyu_finger_triple0.urdf (robot description, URDF)
Before this commit: robot nyu_finger0, 6 links, 5 joints
Links:
- link finger0_base_link: geometry collision mesh filename=package://mim_robots/robots/trifinger/meshes/base_back.stl scale=1 1 1; collision mesh filename=package://mim_robots/robots/trifinger/meshes/base_front.stl scale=1 1 1
- link finger0_lower_link: geometry collision mesh filename=package://mim_robots/robots/trifinger/meshes/lower_link.stl scale=1 1 1; visual mesh filename=package://mim_robots/robots/trifinger/meshes/lower_link.stl scale=1 1 1
- link finger0_middle_link: geometry collision mesh filename=package://mim_robots/robots/trifinger/meshes/middle_link.stl scale=1 1 1; visual mesh filename=package://mim_robots/robots/trifinger/meshes/middle_link.stl scale=1 1 1
- link finger0_upper_link: geometry collision mesh filename=package://mim_robots/robots/trifinger/meshes/upper_link.stl scale=1 1 1; visual mesh filename=package://mim_robots/robots/trifinger/meshes/upper_link.stl scale=1 1 1

File: robots/trifinger/nyu_finger_triple1.urdf (robot description, URDF)
Before this commit: robot nyu_finger1, 6 links, 5 joints
Links:
- link finger1_base_link: geometry collision mesh filename=package://mim_robots/robots/trifinger/meshes/base_back.stl scale=1 1 1; collision mesh filename=package://mim_robots/robots/trifinger/meshes/base_front.stl scale=1 1 1
- link finger1_lower_link: geometry collision mesh filename=package://mim_robots/robots/trifinger/meshes/lower_link.stl scale=1 1 1; visual mesh filename=package://mim_robots/robots/trifinger/meshes/lower_link.stl scale=1 1 1
- link finger1_middle_link: geometry collision mesh filename=package://mim_robots/robots/trifinger/meshes/middle_link.stl scale=1 1 1; visual mesh filename=package://mim_robots/robots/trifinger/meshes/middle_link.stl scale=1 1 1
- link finger1_upper_link: geometry collision mesh filename=package://mim_robots/robots/trifinger/meshes/upper_link.stl scale=1 1 1; visual mesh filename=package://mim_robots/robots/trifinger/meshes/upper_link.stl scale=1 1 1

File: robots/trifinger/nyu_finger_triple2.urdf (robot description, URDF)
Before this commit: robot nyu_finger2, 6 links, 5 joints
Links:
- link finger2_base_link: geometry collision mesh filename=package://mim_robots/robots/trifinger/meshes/base_back.stl scale=1 1 1; collision mesh filename=package://mim_robots/robots/trifinger/meshes/base_front.stl scale=1 1 1
- link finger2_lower_link: geometry collision mesh filename=package://mim_robots/robots/trifinger/meshes/lower_link.stl scale=1 1 1; visual mesh filename=package://mim_robots/robots/trifinger/meshes/lower_link.stl scale=1 1 1
- link finger2_middle_link: geometry collision mesh filename=package://mim_robots/robots/trifinger/meshes/middle_link.stl scale=1 1 1; visual mesh filename=package://mim_robots/robots/trifinger/meshes/middle_link.stl scale=1 1 1
- link finger2_upper_link: geometry collision mesh filename=package://mim_robots/robots/trifinger/meshes/upper_link.stl scale=1 1 1; visual mesh filename=package://mim_robots/robots/trifinger/meshes/upper_link.stl scale=1 1 1
