Commit message: make the package pip installable

File: python/mim_robots/robots/kuka/kuka.urdf (robot description, URDF)
Before this commit: robot KUKAiiwa14, 9 links, 8 joints
Links:
- link L1: geometry collision mesh filename=package://kuka/meshes/kuka/iiwa_link_1.stl; visual mesh filename=package://kuka/meshes/kuka/iiwa_link_1.stl
- link L2: geometry collision mesh filename=package://kuka/meshes/kuka/iiwa_link_2.stl; visual mesh filename=package://kuka/meshes/kuka/iiwa_link_2.stl
- link L3: geometry collision mesh filename=package://kuka/meshes/kuka/iiwa_link_3.stl; visual mesh filename=package://kuka/meshes/kuka/iiwa_link_3.stl
- link L4: geometry collision mesh filename=package://kuka/meshes/kuka/iiwa_link_4.stl; visual mesh filename=package://kuka/meshes/kuka/iiwa_link_4.stl
- link L5: geometry collision mesh filename=package://kuka/meshes/kuka/iiwa_link_5.stl; visual mesh filename=package://kuka/meshes/kuka/iiwa_link_5.stl
- link L6: geometry collision mesh filename=package://kuka/meshes/kuka/iiwa_link_6.stl; visual mesh filename=package://kuka/meshes/kuka/iiwa_link_6.stl
- link L7: geometry collision mesh filename=package://kuka/meshes/kuka/iiwa_link_7.stl; visual mesh filename=package://kuka/meshes/kuka/iiwa_link_7.stl
- link iiwa_base: geometry collision mesh filename=package://kuka/meshes/kuka/iiwa_base.stl; visual mesh filename=package://kuka/meshes/kuka/iiwa_base.stl

File: python/mim_robots/robots/kuka/kuka_gripper.urdf (robot description, URDF)
Before this commit: robot KUKAiiwa14, 21 links, 20 joints
Links:
- link L1: geometry collision mesh filename=package://kuka/meshes/kuka/iiwa_link_1.stl; visual mesh filename=package://kuka/meshes/kuka/iiwa_link_1.stl
- link L2: geometry collision mesh filename=package://kuka/meshes/kuka/iiwa_link_2.stl; visual mesh filename=package://kuka/meshes/kuka/iiwa_link_2.stl
- link L3: geometry collision mesh filename=package://kuka/meshes/kuka/iiwa_link_3.stl; visual mesh filename=package://kuka/meshes/kuka/iiwa_link_3.stl
- link L4: geometry collision mesh filename=package://kuka/meshes/kuka/iiwa_link_4.stl; visual mesh filename=package://kuka/meshes/kuka/iiwa_link_4.stl
- link L5: geometry collision mesh filename=package://kuka/meshes/kuka/iiwa_link_5.stl; visual mesh filename=package://kuka/meshes/kuka/iiwa_link_5.stl
- link L6: geometry collision mesh filename=package://kuka/meshes/kuka/iiwa_link_6.stl; visual mesh filename=package://kuka/meshes/kuka/iiwa_link_6.stl
- link L7: geometry collision mesh filename=package://kuka/meshes/kuka/iiwa_link_7.stl; visual mesh filename=package://kuka/meshes/kuka/iiwa_link_7.stl
- link iiwa_base: geometry collision mesh filename=package://kuka/meshes/kuka/iiwa_base.stl; visual mesh filename=package://kuka/meshes/kuka/iiwa_base.stl
- link robotiq_2f_85_base: geometry collision mesh filename=package://kuka/meshes/gripper/robotiq-2f-base.obj scale=0.001 0.001 0.001; visual mesh filename=package://kuka/meshes/gripper/robotiq-2f-base.obj scale=0.1 0.1 0.1
- link robotiq_2f_85_left_coupler: geometry collision mesh filename=package://kuka/meshes/gripper/robotiq-2f-coupler.obj scale=0.001 0.001 0.001; visual mesh filename=package://kuka/meshes/gripper/robotiq-2f-coupler.obj scale=0.1 0.1 0.1
- link robotiq_2f_85_left_driver: geometry collision mesh filename=package://kuka/meshes/gripper/robotiq-2f-driver.obj scale=0.001 0.001 0.001; visual mesh filename=package://kuka/meshes/gripper/robotiq-2f-driver.obj scale=0.1 0.1 0.1
- link robotiq_2f_85_left_follower: geometry collision mesh filename=package://kuka/meshes/gripper/robotiq-2f-follower.obj scale=0.001 0.001 0.001; visual mesh filename=package://kuka/meshes/gripper/robotiq-2f-follower.obj scale=0.1 0.1 0.1
- link robotiq_2f_85_left_pad: geometry collision mesh filename=package://kuka/meshes/gripper/robotiq-2f-pad.stl scale=0.001 0.001 0.001; visual mesh filename=package://kuka/meshes/gripper/robotiq-2f-pad.stl scale=0.0001 0.0001 0.0001
- link robotiq_2f_85_left_spring_link: geometry collision mesh filename=package://kuka/meshes/gripper/robotiq-2f-spring_link.obj scale=0.001 0.001 0.001; visual mesh filename=package://kuka/meshes/gripper/robotiq-2f-spring_link.obj scale=0.1 0.1 0.1
- link robotiq_2f_85_right_coupler: geometry collision mesh filename=package://kuka/meshes/gripper/robotiq-2f-coupler.obj scale=0.001 0.001 0.001; visual mesh filename=package://kuka/meshes/gripper/robotiq-2f-coupler.obj scale=0.1 0.1 0.1
- link robotiq_2f_85_right_driver: geometry collision mesh filename=package://kuka/meshes/gripper/robotiq-2f-driver.obj scale=0.001 0.001 0.001; visual mesh filename=package://kuka/meshes/gripper/robotiq-2f-driver.obj scale=0.1 0.1 0.1
- link robotiq_2f_85_right_follower: geometry collision mesh filename=package://kuka/meshes/gripper/robotiq-2f-follower.obj scale=0.001 0.001 0.001; visual mesh filename=package://kuka/meshes/gripper/robotiq-2f-follower.obj scale=0.1 0.1 0.1
- link robotiq_2f_85_right_pad: geometry collision mesh filename=package://kuka/meshes/gripper/robotiq-2f-pad.stl scale=0.001 0.001 0.001; visual mesh filename=package://kuka/meshes/gripper/robotiq-2f-pad.stl scale=0.0001 0.0001 0.0001
- link robotiq_2f_85_right_spring_link: geometry collision mesh filename=package://kuka/meshes/gripper/robotiq-2f-spring_link.obj scale=0.001 0.001 0.001; visual mesh filename=package://kuka/meshes/gripper/robotiq-2f-spring_link.obj scale=0.1 0.1 0.1

File: python/mim_robots/robots/teststand/teststand.urdf (robot description, URDF)
Before this commit: robot teststand, 5 links, 4 joints
Links:
- link base_link: geometry collision box size=0.2 0.1 0.1; visual mesh filename=package://teststand/meshes/cube.obj scale=0.2 0.1 0.1
- link contact: geometry collision mesh filename=package://teststand/meshes/solo_foot.stl; visual mesh filename=package://teststand/meshes/solo_foot.stl
- link shank: geometry collision mesh filename=package://teststand/meshes/solo_lower_leg_left_side.stl; visual mesh filename=package://teststand/meshes/solo_lower_leg_left_side.stl
- link upperleg: geometry collision mesh filename=package://teststand/meshes/solo_upper_leg_left_side.stl; visual mesh filename=package://teststand/meshes/solo_upper_leg_left_side.stl

File: python/mim_robots/robots/trifinger/nyu_finger_triple0.urdf (robot description, URDF)
Before this commit: robot nyu_finger1, 6 links, 5 joints
Links:
- removed link finger1_base_link
- removed link finger1_lower_link
- removed link finger1_middle_link
- removed link finger1_tip_link
- removed link finger1_upper_link
- added link finger0_base_link, mass 1; collision mesh filename=package://trifinger/meshes/base_back.stl scale=1 1 1; collision mesh filename=package://trifinger/meshes/base_front.stl scale=1 1 1
- added link finger0_lower_link, mass 0.03070; collision mesh filename=package://trifinger/meshes/lower_link.stl scale=1 1 1; visual mesh filename=package://trifinger/meshes/lower_link.stl scale=1 1 1
- added link finger0_middle_link, mass 0.14854; collision mesh filename=package://trifinger/meshes/middle_link.stl scale=1 1 1; visual mesh filename=package://trifinger/meshes/middle_link.stl scale=1 1 1
- added link finger0_tip_link, mass 0.01
- added link finger0_upper_link, mass 0.14854; collision mesh filename=package://trifinger/meshes/upper_link.stl scale=1 1 1; visual mesh filename=package://trifinger/meshes/upper_link.stl scale=1 1 1
Joints:
- removed joint base_to_finger1
- removed joint finger1_base_to_upper_joint
- removed joint finger1_lower_to_tip_joint
- removed joint finger1_middle_to_lower_joint
- removed joint finger1_upper_to_middle_joint
- added joint base_to_finger0: type fixed, parent base_link, child finger0_base_link, origin xyz=-0.065 0 0.37
- added joint finger0_base_to_upper_joint: type revolute, parent finger0_base_link, child finger0_upper_link, origin xyz=0 0 0 rpy=0 0 0, axis -1 0 0, limit lower=-1.57079632679 upper=1.57079632679 effort=1000 velocity=1000
- added joint finger0_lower_to_tip_joint: type fixed, parent finger0_lower_link, child finger0_tip_link, origin xyz=0 -0.008 -0.16
- added joint finger0_middle_to_lower_joint: type revolute, parent finger0_middle_link, child finger0_lower_link, origin xyz=0 -0.03745 -0.16 rpy=0 0 0, axis 0 1 0, limit lower=-3.14159265359 upper=3.14159265359 effort=1000 velocity=1000
- added joint finger0_upper_to_middle_joint: type revolute, parent finger0_upper_link, child finger0_middle_link, origin xyz=0 -0.014 0 rpy=0 0 0, axis 0 1 0, limit lower=-1.57079632679 upper=1.57079632679 effort=1000 velocity=1000

File: python/mim_robots/robots/trifinger/nyu_finger_triple1.urdf (robot description, URDF)
Before this commit: robot nyu_finger0, 6 links, 5 joints
Links:
- removed link finger0_base_link
- removed link finger0_lower_link
- removed link finger0_middle_link
- removed link finger0_tip_link
- removed link finger0_upper_link
- added link finger1_base_link, mass 1; collision mesh filename=package://trifinger/meshes/base_back.stl scale=1 1 1; collision mesh filename=package://trifinger/meshes/base_front.stl scale=1 1 1
- added link finger1_lower_link, mass 0.03070; collision mesh filename=package://trifinger/meshes/lower_link.stl scale=1 1 1; visual mesh filename=package://trifinger/meshes/lower_link.stl scale=1 1 1
- added link finger1_middle_link, mass 0.14854; collision mesh filename=package://trifinger/meshes/middle_link.stl scale=1 1 1; visual mesh filename=package://trifinger/meshes/middle_link.stl scale=1 1 1
- added link finger1_tip_link, mass 0.01
- added link finger1_upper_link, mass 0.14854; collision mesh filename=package://trifinger/meshes/upper_link.stl scale=1 1 1; visual mesh filename=package://trifinger/meshes/upper_link.stl scale=1 1 1
Joints:
- removed joint base_to_finger0
- removed joint finger0_base_to_upper_joint
- removed joint finger0_lower_to_tip_joint
- removed joint finger0_middle_to_lower_joint
- removed joint finger0_upper_to_middle_joint
- added joint base_to_finger1: type fixed, parent base_link, child finger1_base_link, origin xyz=0.0325 -0.0563 0.37 rpy=0 0 2.09
- added joint finger1_base_to_upper_joint: type revolute, parent finger1_base_link, child finger1_upper_link, origin xyz=0 0 0 rpy=0 0 0, axis -1 0 0, limit lower=-1.57079632679 upper=1.57079632679 effort=1000 velocity=1000
- added joint finger1_lower_to_tip_joint: type fixed, parent finger1_lower_link, child finger1_tip_link, origin xyz=0 -0.008 -0.16
- added joint finger1_middle_to_lower_joint: type revolute, parent finger1_middle_link, child finger1_lower_link, origin xyz=0 -0.03745 -0.16 rpy=0 0 0, axis 0 1 0, limit lower=-3.14159265359 upper=3.14159265359 effort=1000 velocity=1000
- added joint finger1_upper_to_middle_joint: type revolute, parent finger1_upper_link, child finger1_middle_link, origin xyz=0 -0.014 0 rpy=0 0 0, axis 0 1 0, limit lower=-1.57079632679 upper=1.57079632679 effort=1000 velocity=1000

File: python/mim_robots/robots/trifinger/nyu_finger_triple2.urdf (robot description, URDF)
Before this commit: robot nyu_finger2, 6 links, 5 joints
Links:
- link finger2_base_link: geometry collision mesh filename=package://trifinger/meshes/base_back.stl scale=1 1 1; collision mesh filename=package://trifinger/meshes/base_front.stl scale=1 1 1
- link finger2_lower_link: geometry collision mesh filename=package://trifinger/meshes/lower_link.stl scale=1 1 1; visual mesh filename=package://trifinger/meshes/lower_link.stl scale=1 1 1
- link finger2_middle_link: geometry collision mesh filename=package://trifinger/meshes/middle_link.stl scale=1 1 1; visual mesh filename=package://trifinger/meshes/middle_link.stl scale=1 1 1
- link finger2_upper_link: geometry collision mesh filename=package://trifinger/meshes/upper_link.stl scale=1 1 1; visual mesh filename=package://trifinger/meshes/upper_link.stl scale=1 1 1
