Commit message: finished xmls for kuka and teststand

File: python/mim_robots/robots/kuka/urdf/iiwa_ft_sensor_ball.urdf (robot description, URDF)
Before this commit: robot KUKAiiwa14, 14 links, 13 joints
Links:
- link ball_transfer: geometry collision mesh filename=package://robot_properties_kuka/meshes/5674K57_flange_mount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 scale=0.0254 0.0254 0.0254; visual mesh filename=package://robot_properties_kuka/meshes/5674K57_flange_mount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 scale=0.0254 0.0254 0.0254
