Commit message: finished implementing robot loaders

File: python/mim_robots/robots/kuka/urdf/iiwa.urdf (robot description, URDF)
Before this commit: robot KUKAiiwa14, 10 links, 9 joints
Links:
- link L1: geometry collision mesh filename=iiwa_link_1.stl; visual mesh filename=iiwa_link_1.stl
- link L2: geometry collision mesh filename=iiwa_link_2.stl; visual mesh filename=iiwa_link_2.stl
- link L3: geometry collision mesh filename=iiwa_link_3.stl; visual mesh filename=iiwa_link_3.stl
- link L4: geometry collision mesh filename=iiwa_link_4.stl; visual mesh filename=iiwa_link_4.stl
- link L5: geometry collision mesh filename=iiwa_link_5.stl; visual mesh filename=iiwa_link_5.stl
- link L6: geometry collision mesh filename=iiwa_link_6.stl; visual mesh filename=iiwa_link_6.stl
- link L7: geometry collision mesh filename=iiwa_link_7.stl; visual mesh filename=iiwa_link_7.stl
- link contact: geometry collision mesh filename=tennis_ball_smaller.obj; visual mesh filename=tennis_ball_smaller.obj
- link iiwa_base: geometry collision mesh filename=iiwa_base.stl; visual mesh filename=iiwa_base.stl

Commit message: replaced IiwaConfig dependency by RobotInfo in iiwaWrapper

File: python/mim_robots/robots/kuka/urdf/iiwa.urdf (robot description, URDF)
Before this commit: robot KUKAiiwa14, 10 links, 9 joints
Links:
- link L1: geometry collision mesh filename=package://meshes/kuka/iiwa_link_1.stl; visual mesh filename=package://meshes/kuka/iiwa_link_1.stl
- link L2: geometry collision mesh filename=package://meshes/kuka/iiwa_link_2.stl; visual mesh filename=package://meshes/kuka/iiwa_link_2.stl
- link L3: geometry collision mesh filename=package://meshes/kuka/iiwa_link_3.stl; visual mesh filename=package://meshes/kuka/iiwa_link_3.stl
- link L4: geometry collision mesh filename=package://meshes/kuka/iiwa_link_4.stl; visual mesh filename=package://meshes/kuka/iiwa_link_4.stl
- link L5: geometry collision mesh filename=package://meshes/kuka/iiwa_link_5.stl; visual mesh filename=package://meshes/kuka/iiwa_link_5.stl
- link L6: geometry collision mesh filename=package://meshes/kuka/iiwa_link_6.stl; visual mesh filename=package://meshes/kuka/iiwa_link_6.stl
- link L7: geometry collision mesh filename=package://meshes/kuka/iiwa_link_7.stl; visual mesh filename=package://meshes/kuka/iiwa_link_7.stl
- link contact: geometry collision mesh filename=package://meshes/kuka/tennis_ball_smaller.obj; visual mesh filename=package://meshes/kuka/tennis_ball_smaller.obj
- link iiwa_base: geometry collision mesh filename=package://meshes/kuka/iiwa_base.stl; visual mesh filename=package://meshes/kuka/iiwa_base.stl

File: python/mim_robots/robots/kuka/urdf/iiwa_ft_sensor_ball.urdf (robot description, URDF)
Before this commit: robot KUKAiiwa14, 14 links, 13 joints
Links:
- link L1: geometry collision mesh filename=package://meshes/kuka/iiwa_link_1.stl; visual mesh filename=package://meshes/kuka/iiwa_link_1.stl
- link L2: geometry collision mesh filename=package://meshes/kuka/iiwa_link_2.stl; visual mesh filename=package://meshes/kuka/iiwa_link_2.stl
- link L3: geometry collision mesh filename=package://meshes/kuka/iiwa_link_3.stl; visual mesh filename=package://meshes/kuka/iiwa_link_3.stl
- link L4: geometry collision mesh filename=package://meshes/kuka/iiwa_link_4.stl; visual mesh filename=package://meshes/kuka/iiwa_link_4.stl
- link L5: geometry collision mesh filename=package://meshes/kuka/iiwa_link_5.stl; visual mesh filename=package://meshes/kuka/iiwa_link_5.stl
- link L6: geometry collision mesh filename=package://meshes/kuka/iiwa_link_6.stl; visual mesh filename=package://meshes/kuka/iiwa_link_6.stl
- link L7: geometry collision mesh filename=package://meshes/kuka/iiwa_link_7.stl; visual mesh filename=package://meshes/kuka/iiwa_link_7.stl
- link ball_transfer: geometry collision mesh filename=package://meshes/kuka/5674K57_flange_mount_ball_transfer.stl scale=0.0254 0.0254 0.0254; visual mesh filename=package://meshes/kuka/5674K57_flange_mount_ball_transfer.stl scale=0.0254 0.0254 0.0254
- link iiwa_base: geometry collision mesh filename=package://meshes/kuka/iiwa_base.stl; visual mesh filename=package://meshes/kuka/iiwa_base.stl
- link kuka_to_sensor_mount: geometry collision mesh filename=package://meshes/kuka/kuka_to_sensor_mount.stl scale=0.001 0.001 0.001; visual mesh filename=package://meshes/kuka/kuka_to_sensor_mount.stl scale=0.001 0.001 0.001
- link sensor_to_case_mount: geometry collision mesh filename=package://meshes/kuka/sensor_to_case_mount.stl scale=0.001 0.001 0.001; visual mesh filename=package://meshes/kuka/sensor_to_case_mount.stl scale=0.001 0.001 0.001

File: python/mim_robots/robots/kuka/urdf/iiwa_ft_sensor_shell.urdf (robot description, URDF)
Before this commit: robot KUKAiiwa14, 11 links, 10 joints
Links:
- link L1: geometry collision mesh filename=package://meshes/kuka/iiwa_link_1.stl; visual mesh filename=package://meshes/kuka/iiwa_link_1.stl
- link L2: geometry collision mesh filename=package://meshes/kuka/iiwa_link_2.stl; visual mesh filename=package://meshes/kuka/iiwa_link_2.stl
- link L3: geometry collision mesh filename=package://meshes/kuka/iiwa_link_3.stl; visual mesh filename=package://meshes/kuka/iiwa_link_3.stl
- link L4: geometry collision mesh filename=package://meshes/kuka/iiwa_link_4.stl; visual mesh filename=package://meshes/kuka/iiwa_link_4.stl
- link L5: geometry collision mesh filename=package://meshes/kuka/iiwa_link_5.stl; visual mesh filename=package://meshes/kuka/iiwa_link_5.stl
- link L6: geometry collision mesh filename=package://meshes/kuka/iiwa_link_6.stl; visual mesh filename=package://meshes/kuka/iiwa_link_6.stl
- link L7: geometry collision mesh filename=package://meshes/kuka/iiwa_link_7.stl; visual mesh filename=package://meshes/kuka/iiwa_link_7.stl
- link assembled_ee: geometry collision mesh filename=package://meshes/kuka/assembled_ee.stl scale=0.001 0.001 0.001; visual mesh filename=package://meshes/kuka/assembled_ee.stl scale=0.001 0.001 0.001
- link iiwa_base: geometry collision mesh filename=package://meshes/kuka/iiwa_base.stl; visual mesh filename=package://meshes/kuka/iiwa_base.stl
