Commit message: added gripper + tested in bullet

File: python/mim_robots/robots/kuka/urdf/iiwa_gripper.urdf (robot description, URDF)
Before this commit: robot KUKAiiwa14, 21 links, 20 joints
Links:
- link L1: geometry collision mesh filename=package://meshes/kuka/iiwa_link_1.stl; visual mesh filename=package://meshes/kuka/iiwa_link_1.stl
- link L2: geometry collision mesh filename=package://meshes/kuka/iiwa_link_2.stl; visual mesh filename=package://meshes/kuka/iiwa_link_2.stl
- link L3: geometry collision mesh filename=package://meshes/kuka/iiwa_link_3.stl; visual mesh filename=package://meshes/kuka/iiwa_link_3.stl
- link L4: geometry collision mesh filename=package://meshes/kuka/iiwa_link_4.stl; visual mesh filename=package://meshes/kuka/iiwa_link_4.stl
- link L5: geometry collision mesh filename=package://meshes/kuka/iiwa_link_5.stl; visual mesh filename=package://meshes/kuka/iiwa_link_5.stl
- link L6: geometry collision mesh filename=package://meshes/kuka/iiwa_link_6.stl; visual mesh filename=package://meshes/kuka/iiwa_link_6.stl
- link L7: geometry collision mesh filename=package://meshes/kuka/iiwa_link_7.stl; visual mesh filename=package://meshes/kuka/iiwa_link_7.stl
- link iiwa_base: geometry collision mesh filename=package://meshes/kuka/iiwa_base.stl; visual mesh filename=package://meshes/kuka/iiwa_base.stl
- link robotiq_2f_85_base: geometry collision mesh filename=package://meshes/gripper/robotiq-2f-base.obj scale=0.001 0.001 0.001; visual mesh filename=package://meshes/gripper/robotiq-2f-base.obj scale=0.1 0.1 0.1
- link robotiq_2f_85_left_coupler: geometry collision mesh filename=package://meshes/gripper/robotiq-2f-coupler.obj scale=0.001 0.001 0.001; visual mesh filename=package://meshes/gripper/robotiq-2f-coupler.obj scale=0.1 0.1 0.1
- link robotiq_2f_85_left_driver: geometry collision mesh filename=package://meshes/gripper/robotiq-2f-driver.obj scale=0.001 0.001 0.001; visual mesh filename=package://meshes/gripper/robotiq-2f-driver.obj scale=0.1 0.1 0.1
- link robotiq_2f_85_left_follower: geometry collision mesh filename=package://meshes/gripper/robotiq-2f-follower.obj scale=0.001 0.001 0.001; visual mesh filename=package://meshes/gripper/robotiq-2f-follower.obj scale=0.1 0.1 0.1
- link robotiq_2f_85_left_pad: geometry collision mesh filename=package://meshes/gripper/robotiq-2f-pad.stl scale=0.001 0.001 0.001; visual mesh filename=package://meshes/gripper/robotiq-2f-pad.stl scale=0.0001 0.0001 0.0001
- link robotiq_2f_85_left_spring_link: geometry collision mesh filename=package://meshes/gripper/robotiq-2f-spring_link.obj scale=0.001 0.001 0.001; visual mesh filename=package://meshes/gripper/robotiq-2f-spring_link.obj scale=0.1 0.1 0.1
- link robotiq_2f_85_right_coupler: geometry collision mesh filename=package://meshes/gripper/robotiq-2f-coupler.obj scale=0.001 0.001 0.001; visual mesh filename=package://meshes/gripper/robotiq-2f-coupler.obj scale=0.1 0.1 0.1
- link robotiq_2f_85_right_driver: geometry collision mesh filename=package://meshes/gripper/robotiq-2f-driver.obj scale=0.001 0.001 0.001; visual mesh filename=package://meshes/gripper/robotiq-2f-driver.obj scale=0.1 0.1 0.1
- link robotiq_2f_85_right_follower: geometry collision mesh filename=package://meshes/gripper/robotiq-2f-follower.obj scale=0.001 0.001 0.001; visual mesh filename=package://meshes/gripper/robotiq-2f-follower.obj scale=0.1 0.1 0.1
- link robotiq_2f_85_right_pad: geometry collision mesh filename=package://meshes/gripper/robotiq-2f-pad.stl scale=0.001 0.001 0.001; visual mesh filename=package://meshes/gripper/robotiq-2f-pad.stl scale=0.0001 0.0001 0.0001
- link robotiq_2f_85_right_spring_link: geometry collision mesh filename=package://meshes/gripper/robotiq-2f-spring_link.obj scale=0.001 0.001 0.001; visual mesh filename=package://meshes/gripper/robotiq-2f-spring_link.obj scale=0.1 0.1 0.1
Joints:
- removed joint base_link_robotiq_2f_85_base_joint
- added joint EE: type fixed, parent L7, child robotiq_2f_85_base, origin xyz=0 0 0 rpy=0 0 0
