Commit message: added capsule on ft sensor mounting piece

File: python/mim_robots/robots/kuka/urdf/iiwa_convex_ft_sensor_shell.urdf (robot description, URDF)
Before this commit: robot KUKAiiwa14, 11 links, 10 joints
Links:
- link assembled_ee: geometry collision cylinder length=0.1 radius=0.04; visual mesh filename=package://meshes/kuka/assembled_ee.stl scale=0.001 0.001 0.001

Commit message: tuned capsule size on FT shell end-effector

File: python/mim_robots/robots/kuka/urdf/iiwa_convex_ft_sensor_shell.urdf (robot description, URDF)
Before this commit: robot KUKAiiwa14, 11 links, 10 joints
Links:
- link assembled_ee: geometry collision cylinder length=0.1 radius=0.01; visual mesh filename=package://meshes/kuka/assembled_ee.stl scale=0.001 0.001 0.001

Commit message: increased size of eft end-eff capsule

File: python/mim_robots/robots/kuka/urdf/iiwa_convex_ft_sensor_shell.urdf (robot description, URDF)
Before this commit: robot KUKAiiwa14, 11 links, 10 joints
Links:
- link assembled_ee: geometry collision cylinder length=0.3 radius=0.06; visual mesh filename=package://meshes/kuka/assembled_ee.stl scale=0.001 0.001 0.001
