Commit message: fixed solo meshes path

File: python/mim_robots/robots/solo12/urdf/solo12.urdf (robot description, URDF)
Before this commit: robot solo, 17 links, 16 joints
Links:
- link FL_LOWER_LEG: geometry collision mesh filename=package://meshes/solo_lower_leg_v2_left_side.stl; visual mesh filename=package://meshes/solo_lower_leg_v2_left_side.stl
- link FL_SHOULDER: geometry collision mesh filename=package://meshes/solo12_hip_fe_fl.stl; visual mesh filename=package://meshes/solo12_hip_fe_fl.stl
- link FL_UPPER_LEG: geometry collision mesh filename=package://meshes/solo_upper_leg_left_side.stl; visual mesh filename=package://meshes/solo_upper_leg_left_side.stl
- link FR_LOWER_LEG: geometry collision mesh filename=package://meshes/solo_lower_leg_v2_right_side.stl; visual mesh filename=package://meshes/solo_lower_leg_v2_right_side.stl
- link FR_SHOULDER: geometry collision mesh filename=package://meshes/solo12_hip_fe_fr.stl; visual mesh filename=package://meshes/solo12_hip_fe_fr.stl
- link FR_UPPER_LEG: geometry collision mesh filename=package://meshes/solo_upper_leg_right_side.stl; visual mesh filename=package://meshes/solo_upper_leg_right_side.stl
- link HL_LOWER_LEG: geometry collision mesh filename=package://meshes/solo_lower_leg_v2_left_side.stl; visual mesh filename=package://meshes/solo_lower_leg_v2_left_side.stl
- link HL_SHOULDER: geometry collision mesh filename=package://meshes/solo12_hip_fe_hl.stl; visual mesh filename=package://meshes/solo12_hip_fe_hl.stl
- link HL_UPPER_LEG: geometry collision mesh filename=package://meshes/solo_upper_leg_left_side.stl; visual mesh filename=package://meshes/solo_upper_leg_left_side.stl
- link HR_LOWER_LEG: geometry collision mesh filename=package://meshes/solo_lower_leg_v2_right_side.stl; visual mesh filename=package://meshes/solo_lower_leg_v2_right_side.stl
- link HR_SHOULDER: geometry collision mesh filename=package://meshes/solo12_hip_fe_hr.stl; visual mesh filename=package://meshes/solo12_hip_fe_hr.stl
- link HR_UPPER_LEG: geometry collision mesh filename=package://meshes/solo_upper_leg_right_side.stl; visual mesh filename=package://meshes/solo_upper_leg_right_side.stl
- link base_link: geometry collision mesh filename=package://meshes/solo_12_base.stl; visual mesh filename=package://meshes/solo_12_base.stl
