Commit message: added working mujoco demo

File: python/mim_robots/robots/teststand/urdf/teststand.urdf (robot description, URDF)
Before this commit: robot teststand, 5 links, 4 joints
Links:
- link base_link: geometry collision box size=0.2 0.1 0.1; visual mesh filename=../meshes/cube.obj scale=0.2 0.1 0.1
- link contact: geometry collision mesh filename=../meshes/solo_foot.stl; visual mesh filename=../meshes/solo_foot.stl
- link shank: geometry collision mesh filename=../meshes/solo_lower_leg_left_side.stl; visual mesh filename=../meshes/solo_lower_leg_left_side.stl
- link upperleg: geometry collision mesh filename=../meshes/solo_upper_leg_left_side.stl; visual mesh filename=../meshes/solo_upper_leg_left_side.stl

Commit message: fixed mesh path in teststand urdf

File: python/mim_robots/robots/teststand/urdf/teststand.urdf (robot description, URDF)
Before this commit: robot teststand, 5 links, 4 joints
Links:
- link base_link: geometry collision box size=0.2 0.1 0.1; visual mesh filename=package://meshes/cube.obj scale=0.2 0.1 0.1
- link contact: geometry collision mesh filename=package://meshes/solo_foot.stl; visual mesh filename=package://meshes/solo_foot.stl
- link shank: geometry collision mesh filename=package://meshes/solo_lower_leg_left_side.stl; visual mesh filename=package://meshes/solo_lower_leg_left_side.stl
- link upperleg: geometry collision mesh filename=package://meshes/solo_upper_leg_left_side.stl; visual mesh filename=package://meshes/solo_upper_leg_left_side.stl
