Commit message: Fix bullet simulation

File: python/mim_robots/robots/panda/urdf/panda.urdf (robot description, URDF)
Before this commit: robot panda, 14 links, 13 joints
Joints:
- removed joint panda_contact_joint2
- added joint panda_contact_joint: type fixed, parent panda_hand, child contact, origin xyz=0 0 0.0584 rpy=0 0 0

Commit message: Convert visual meshes to STL

File: python/mim_robots/robots/panda/urdf/panda.urdf (robot description, URDF)
Before this commit: robot panda, 14 links, 13 joints
Links:
- link panda_hand: geometry collision mesh filename=package://meshes/collision/hand.stl; visual mesh filename=package://meshes/visual/hand.stl
- link panda_leftfinger: geometry collision box size=17.5e-3 15.2e-3 18.5e-3; collision box size=17.5e-3 7e-3 23.5e-3
- link panda_link0: geometry collision mesh filename=package://meshes/collision/link0.stl; visual mesh filename=package://meshes/visual/link0.stl
- link panda_link1: geometry collision mesh filename=package://meshes/collision/link1.stl; visual mesh filename=package://meshes/visual/link1.stl
- link panda_link2: geometry collision mesh filename=package://meshes/collision/link2.stl; visual mesh filename=package://meshes/visual/link2.stl
- link panda_link3: geometry collision mesh filename=package://meshes/collision/link3.stl; visual mesh filename=package://meshes/visual/link3.stl
- link panda_link4: geometry collision mesh filename=package://meshes/collision/link4.stl; visual mesh filename=package://meshes/visual/link4.stl
- link panda_link5: geometry collision mesh filename=package://meshes/collision/link5.stl; visual mesh filename=package://meshes/visual/link5.stl
- link panda_link6: geometry collision mesh filename=package://meshes/collision/link6.stl; visual mesh filename=package://meshes/visual/link6.stl
- link panda_link7: geometry collision mesh filename=package://meshes/collision/link7.stl; visual mesh filename=package://meshes/visual/link7.stl
- link panda_rightfinger: geometry collision box size=17.5e-3 15.2e-3 18.5e-3; collision box size=17.5e-3 7e-3 23.5e-3
