Commit message: cleaned up pinbullet  wrapper joint mapping + go2 wrapper + inertias in go2 urdf

File: python/mim_robots/robots/go2/urdf/go2_with_arm.urdf (robot description, URDF)
Before this commit: robot go2, 37 links, 36 joints
Links:
- link FL_KFElower: mass None -> 0.001
- link FL_KFElower1: mass None -> 0.04
- link FR_KFElower: mass None -> 0.001
- link FR_KFElower1: mass None -> 0.04
- link HL_KFElower: mass None -> 0.001
- link HL_KFElower1: mass None -> 0.04
- link HR_KFElower: mass None -> 0.001
- link HR_KFElower1: mass None -> 0.04
- link ef_tip: mass None -> 0.04
Joints:
- joint Joint1: limit lower=-2.35 upper=2.35 effort=0 velocity=0 -> lower=-2.35 upper=2.35 effort=100 velocity=100
- joint Joint2: limit lower=-1.57 upper=1.57 effort=0 velocity=0 -> lower=-1.57 upper=1.57 effort=100 velocity=100
- joint Joint3: limit lower=-1.57 upper=1.57 effort=0 velocity=0 -> lower=-1.57 upper=1.57 effort=100 velocity=100
- joint Joint4: limit lower=-2.35 upper=2.35 effort=0 velocity=0 -> lower=-2.35 upper=2.35 effort=100 velocity=100
- joint Joint5: limit lower=-1.57 upper=1.57 effort=0 velocity=0 -> lower=-1.57 upper=1.57 effort=100 velocity=100
- joint Joint6: limit lower=-2.35 upper=2.35 effort=0 velocity=0 -> lower=-2.35 upper=2.35 effort=100 velocity=100

Commit message: added collisions on arm tip

File: python/mim_robots/robots/go2/urdf/go2_with_arm.urdf (robot description, URDF)
Before this commit: robot go2, 37 links, 36 joints
Links:
- link Link5: geometry collision mesh filename=d1_assets/stl/Link5.STL; visual mesh filename=d1_assets/stl/Link5.STL
- link Link6: geometry collision mesh filename=d1_assets/stl/Link6-new.stl; visual mesh filename=d1_assets/stl/Link6-new.stl
- link ef_tip: geometry collision sphere radius=0.02; visual sphere radius=0.02
